File: kicad-files-components/sensorV2.kicad_pcb (KiCad board)
At the start: 2 copper layers, 100 x 60 mm, 10 parts, among them J1 Jack-DC, SW1 SW_Push, U1 thing, U2 LF356, U3 ESP-M2, U4 LD1117V33

Commit message: Final setup files to main
Parts:
- BT1: footprint MyStuff:Battery -> 4DPrinting:Battery
- J1: footprint MyStuff:charge_port -> 4DPrinting:charge_port
- R1, R2, R3: value R -> TPU; footprint MyStuff:TPU -> 4DPrinting:TPU
- SW1: footprint MyStuff:switch -> 4DPrinting:switch
- U1: value thing -> Wave Gen; footprint MyStuff:for_thing -> 4DPrinting:wave_gen
- U2: footprint MyStuff:dummy_lf356 -> 4DPrinting:custom_lf356
- U3: footprint MyStuff:MODULE_ESP-M2 -> 4DPrinting:MODULE_ESP-M2
- U4: footprint MyStuff:voltage_regulator -> 4DPrinting:voltage_regulator
Connections:
- J1 pad 1: Net-(BT1-Pad2) -> Net-(BT1-Pad1)
- J1 pad 2: Net-(BT1-Pad1) -> Net-(BT1-Pad2)
