File: kicad-files-components/sensorV2.kicad_sch (KiCad schematic)
At the start: 10 parts, among them J1 Jack-DC, SW1 SW_Push, U1 Wave Gen, U2 LF356, U3 ESP-M2, U4 LD1117V33

Commit message: Final setup files to main
Parts:
- BT1: footprint MyStuff:Battery -> 4DPrinting:Battery
- J1: footprint MyStuff:charge_port -> 4DPrinting:charge_port
- R1, R2, R3: footprint MyStuff:TPU -> 4DPrinting:TPU
- SW1: footprint MyStuff:switch -> 4DPrinting:switch
- U1: footprint MyStuff:for_thing -> 4DPrinting:wave_gen
- U2: footprint MyStuff:dummy_lf356 -> 4DPrinting:custom_lf356
- U3: footprint MyStuff:MODULE_ESP-M2 -> 4DPrinting:MODULE_ESP-M2
- U4: footprint MyStuff:voltage_regulator -> 4DPrinting:voltage_regulator
Changed lines of the file:
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@@
       (effects (font (size 1.27 1.27)) (justify left))
     )
-    (property "Footprint" "MyStuff:Battery" (id 2) (at 184.785 79.121 90)
+    (property "Footprint" "4DPrinting:Battery" (id 2) (at 184.785 79.121 90)
       (effects (font (size 1.27 1.27)) hide)
     )
@@
     (property "Reference" "R2" (id 0) (at 106.68 78.74 90))
     (property "Value" "TPU" (id 1) (at 106.68 81.28 90))
-    (property "Footprint" "MyStuff:TPU" (id 2) (at 106.68 86.233 90)
+    (property "Footprint" "4DPrinting:TPU" (id 2) (at 106.68 86.233 90)
       (effects (font (size 1.27 1.27)) hide)
     )
@@
       (effects (font (size 1.27 1.27)) (justify right))
     )
-    (property "Footprint" "MyStuff:for_thing" (id 2) (at 71.755 81.915 0)
+    (property "Footprint" "4DPrinting:wave_gen" (id 2) (at 71.755 81.915 0)
       (effects (font (size 1.27 1.27)) hide)
     )
@@
     (property "Reference" "U2" (id 0) (at 142.24 80.391 0))
     (property "Value" "LF356" (id 1) (at 142.24 82.931 0))
-    (property "Footprint" "MyStuff:dummy_lf356" (id 2) (at 133.985 83.82 0)
+    (property "Footprint" "4DPrinting:custom_lf356" (id 2) (at 133.985 83.82 0)
       (effects (font (size 1.27 1.27)) hide)
     )
@@
     (property "Reference" "R3" (id 0) (at 107.315 90.17 90))
     (property "Value" "TPU" (id 1) (at 107.315 92.71 90))
-    (property "Footprint" "MyStuff:TPU" (id 2) (at 107.315 98.298 90)
+    (property "Footprint" "4DPrinting:TPU" (id 2) (at 107.315 98.298 90)
       (effects (font (size 1.27 1.27)) hide)
     )
@@
     (property "Reference" "U3" (id 0) (at 157.48 89.535 0))
     (property "Value" "ESP-M2" (id 1) (at 157.48 92.075 0))
-    (property "Footprint" "MyStuff:MODULE_ESP-M2" (id 2) (at 157.48 112.395 0)
+    (property "Footprint" "4DPrinting:MODULE_ESP-M2" (id 2) (at 157.48 112.395 0)
       (effects (font (size 1.27 1.27)) (justify bottom) hide)
     )
@@
     (property "Reference" "R1" (id 0) (at 106.68 67.31 90))
     (property "Value" "TPU" (id 1) (at 106.68 69.85 90))
-    (property "Footprint" "MyStuff:TPU" (id 2) (at 106.68 74.803 90)
+    (property "Footprint" "4DPrinting:TPU" (id 2) (at 106.68 74.803 90)
       (effects (font (size 1.27 1.27)) hide)
     )
@@
     (property "Reference" "U4" (id 0) (at 164.465 91.44 0))
     (property "Value" "LD1117V33" (id 1) (at 164.465 88.9 0))
-    (property "Footprint" "MyStuff:voltage_regulator" (id 2) (at 164.465 81.28 0)
+    (property "Footprint" "4DPrinting:voltage_regulator" (id 2) (at 164.465 81.28 0)
       (effects (font (size 1.27 1.27)) (justify bottom) hide)
     )
@@
     (property "Reference" "SW1" (id 0) (at 166.37 60.96 0))
     (property "Value" "SW_Push" (id 1) (at 166.37 63.5 0))
-    (property "Footprint" "MyStuff:switch" (id 2) (at 166.37 64.135 0)
+    (property "Footprint" "4DPrinting:switch" (id 2) (at 166.37 64.135 0)
       (effects (font (size 1.27 1.27)) hide)
     )
@@
       (effects (font (size 1.27 1.27)) (justify right))
     )
-    (property "Footprint" "MyStuff:charge_port" (id 2) (at 205.74 82.296 0)
+    (property "Footprint" "4DPrinting:charge_port" (id 2) (at 205.74 82.296 0)
       (effects (font (size 1.27 1.27)) hide)
     )
@@
     )
     (path "/0314d948-7a4c-4158-89ac-c56eaf763ca6"
-      (reference "BT1") (unit 1) (value "Battery") (footprint "MyStuff:Battery")
+      (reference "BT1") (unit 1) (value "Battery") (footprint "4DPrinting:Battery")
     )
     (path "/ec0cd66d-bda3-4649-bb86-0213326ed10d"
-      (reference "J1") (unit 1) (value "Jack-DC") (footprint "MyStuff:charge_port")
+      (reference "J1") (unit 1) (value "Jack-DC") (footprint "4DPrinting:charge_port")
     )
     (path "/653ec710-1cff-4655-aab8-5fa9652a0533"
-      (reference "R1") (unit 1) (value "TPU") (footprint "MyStuff:TPU")
+      (reference "R1") (unit 1) (value "TPU") (footprint "4DPrinting:TPU")
     )
     (path "/2048883d-9b57-43d5-a072-feb4d5144fef"
-      (reference "R2") (unit 1) (value "TPU") (footprint "MyStuff:TPU")
+      (reference "R2") (unit 1) (value "TPU") (footprint "4DPrinting:TPU")
     )
     (path "/3156c3cb-2f85-4210-a709-535dd30f1f7e"
-      (reference "R3") (unit 1) (value "TPU") (footprint "MyStuff:TPU")
+      (reference "R3") (unit 1) (value "TPU") (footprint "4DPrinting:TPU")
     )
     (path "/929a3b40-f43f-4259-9eb3-22ccb53ab12b"
-      (reference "SW1") (unit 1) (value "SW_Push") (footprint "MyStuff:switch")
+      (reference "SW1") (unit 1) (value "SW_Push") (footprint "4DPrinting:switch")
     )
     (path "/2ecd08e0-a928-45bf-b655-88e848780f5a"
-      (reference "U1") (unit 1) (value "Wave Gen") (footprint "MyStuff:for_thing")
+      (reference "U1") (unit 1) (value "Wave Gen") (footprint "4DPrinting:wave_gen")
     )
     (path "/2fbd4f9d-b4c6-4098-8be0-4376909a2af4"
-      (reference "U2") (unit 1) (value "LF356") (footprint "MyStuff:dummy_lf356")
+      (reference "U2") (unit 1) (value "LF356") (footprint "4DPrinting:custom_lf356")
     )
     (path "/41187e23-e8ef-45d3-a48b-1659be555d1e"
-      (reference "U3") (unit 1) (value "ESP-M2") (footprint "MyStuff:MODULE_ESP-M2")
+      (reference "U3") (unit 1) (value "ESP-M2") (footprint "4DPrinting:MODULE_ESP-M2")
     )
     (path "/8c87cd2e-e85d-498b-a22c-a62eb6078d41"
-      (reference "U4") (unit 1) (value "LD1117V33") (footprint "MyStuff:voltage_regulator")
-    )
-  )
+      (reference "U4") (unit 1) (value "LD1117V33") (footprint "4DPrinting:voltage_regulator")
+    )
+  )
